Commit message: changed hegiht of baselink in osam_arm_urdf.urdf

File: osam_arm_urdf/urdf/osam_arm_urdf.urdf (robot description, URDF)
Before this commit: robot osam_arm_urdf, 11 links, 10 joints
Joints:
- joint base_joint: origin xyz=0.0 0.0 0.0 rpy=0 0 0 -> xyz=0.0 0.0 10.0 rpy=0 0 0

Commit message: Testing

File: osam_arm_urdf/urdf/osam_arm_urdf.urdf (robot description, URDF)
Before this commit: robot osam_arm_urdf, 11 links, 10 joints
Links:
- link base_link: mass 0.70632 -> 0.01
- link link_1: mass 4.9706 -> 0.01
- link link_2: mass 5.3095 -> 0.01
- link link_3: mass 23.526 -> 0.01
- link link_4: mass 14.099 -> 0.01
- link link_5: mass 2.0698 -> 0.01
- link link_6: mass 1.8548 -> 0.01
- link link_7: mass 0.14601 -> 0.01
- link link_8: mass 0.12436 -> 0.01
- link link_9: mass 0.12436 -> 0.01
