Commit message: Working Velocity controller and sending messages to UE5, need to make setup more streamlined

File: moveit_osam_arm_sim_v2/config/gazebo_osam_arm_4_urdf_v2.urdf (robot description, URDF)
Before this commit: robot osam_arm_4_urdf_v2, 11 links, 10 joints
Joints:
- joint joint6: limit lower=-3.14 upper=3.14 effort=111 velocity=0 -> lower=-3.14 upper=3.14 effort=111 velocity=3

File: osam_arm_4_urdf_v2/urdf/osam_arm_4_urdf_v2.urdf (robot description, URDF)
Before this commit: robot osam_arm_4_urdf_v2, 11 links, 10 joints
Joints:
- joint joint6: limit lower=-3.14 upper=3.14 effort=111 velocity=0 -> lower=-3.14 upper=3.14 effort=111 velocity=3
