Commit message: Working velocity control in moveit_osam_arm_sim_v2, just need to add teleop keyboard inputs and clean everything up

File: osam_arm_4_urdf_v2/urdf/osam_arm_4_urdf_v2.urdf (robot description, URDF)
Before this commit: robot osam_arm_4_urdf_v2, 11 links, 10 joints
Links:
- removed link link_7
- added link ee_link, mass 0.01; collision mesh filename=package://osam_arm_4_urdf_v2/meshes/link_7.STL; visual mesh filename=package://osam_arm_4_urdf_v2/meshes/link_7.STL
Joints:
- joint joint6: child link_7 -> ee_link
- joint joint7: parent link_7 -> ee_link
- joint joint8: parent link_7 -> ee_link

Commit message: renamed comms

File: osam_arm_4_urdf_v2/urdf/osam_arm_4_urdf_v2.urdf (robot description, URDF)
Before this commit: robot osam_arm_4_urdf_v2, 11 links, 10 joints
Joints:
- joint joint8: limit lower=-0.04 upper=0 effort=111 velocity=3 -> lower=0.0 upper=0.04 effort=111 velocity=3
